File: pcb_design/power_distributor/power_distributor.sch (EAGLE design)
At the start: 12 parts

Commit message: [PCB/power_distributor] Correcting wrong JST footprint
Parts:
- BATT_BAL: value B4B-ZR -> (none); device con-jst:B4B-ZR -> SparkFun-Connectors:M04POLAR
Connections:
- net BATT_3: now also BATT_BAL.2; no longer BATT_BAL-2.1
- net GND: now also BATT_BAL.1; no longer BATT_BAL-1.1
- net N$2: now also BATT_BAL.3; no longer BATT_BAL-3.1
- net VCC: now also BATT_BAL.4; no longer BATT_BAL-4.1
